File: KiCad/Sensors/Sensors.kicad_pcb (KiCad board)
At the start: 2 copper layers, 45.7 x 22.9 mm, 13 parts, among them J1 BERG 2x6, U1 OPA1641

Commit message: In Progress for board debugging
Issue with East Sensor being investigated
Routing:
- net GND: track 74.6 -> 82.3 mm
Changed lines of the file:
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@@
     (thickness 1.6)
     (drawings 14)
-    (tracks 97)
+    (tracks 101)
     (zones 0)
     (modules 13)
@@
       (padsonsilk false)
       (subtractmaskfromsilk false)
-      (outputformat 1)
+      (outputformat 3)
       (mirror false)
       (drillshape 0)
@@
   (segment (start 123.19 93.39) (end 123.19 86.36) (width 0.25) (layer B.Cu) (net 8))
   (segment (start 124.73 94.93) (end 123.19 93.39) (width 0.25) (layer B.Cu) (net 8))
-  (segment (start 153.54 93.98) (end 153.54 92.58) (width 0.25) (layer F.Cu) (net 8))
-  (segment (start 153.54 92.58) (end 152.4 91.44) (width 0.25) (layer F.Cu) (net 8))
-  (segment (start 152.4 91.44) (end 152.4 91.44) (width 0.25) (layer F.Cu) (net 8))
-  (via (at 152.4 91.44) (size 0.8) (drill 0.4) (layers F.Cu B.Cu) (net 8))
+  (segment (start 153.54 93.98) (end 153.54 96.39) (width 0.25) (layer F.Cu) (net 8))
+  (segment (start 153.54 96.39) (end 153.67 96.52) (width 0.25) (layer F.Cu) (net 8))
+  (segment (start 152.4 91.44) (end 153.67 91.44) (width 0.25) (layer B.Cu) (net 8))
+  (segment (start 153.67 91.44) (end 154.94 92.71) (width 0.25) (layer B.Cu) (net 8))
+  (segment (start 154.94 92.71) (end 154.94 96.52) (width 0.25) (layer B.Cu) (net 8))
+  (segment (start 154.94 96.52) (end 153.67 96.52) (width 0.25) (layer B.Cu) (net 8))
+  (segment (start 153.67 96.52) (end 153.67 96.52) (width 0.25) (layer B.Cu) (net 8))
+  (via (at 153.67 96.52) (size 0.8) (drill 0.4) (layers F.Cu B.Cu) (net 8))
   (segment (start 149.86 81.28) (end 149.86 81.28) (width 0.25) (layer F.Cu) (net 10))
   (segment (start 148.2575 81.28) (end 149.86 81.28) (width 0.25) (layer F.Cu) (net 10))
